File: nonSNES.kicad_sch (KiCad schematic)
At the start: 399 parts, among them J1 Jack-DC, J3 Conn_02x06_Odd_Even, J4 CONTROLLER 1, J5 CONTROLLER 2, P1 CASSETTE, P2 JST 11FE-BT-VK-N, P3 Conn_01x02_Pin, P7 JST 11FE-BT-VK-N, Q10 C2412K, Q11 C2412K, Q12 C2412K, Q13 C2412K, Q14 C2412K, Q15 C2412K, Q16 C2412K, Q17 C2412K, Q18 2SC5658, Q3 C2412K, Q4 C2412K, Q5 C2412K, Q6 C2412K, Q7 C2412K, Q8 C2412K, Q9 C2412K, SW1 SW_Push, T1 L_Coupled, U1 CPU, U10 LM324, U11 LM809, U12 L7805, U13 S-SMP, U14 S-DSP, U15 MS62256CL-10FC, U16 MS62256CL-10FC, U17 uPD6376, U18 S-CLK, U2 PPU1, U3 PPU2, U4 MS62256CL-10FC, U5 MS62256CL-10FC, U6 WRAM, U7 S-ENC, U8 CIC, X1 17.734MHz, X2 24.576MHz

Commit message: add back old reset switch
Parts:
- added SW2: Old, SNES_Library:ResetSwitch, symbol Switch:SW_Push
- SW1: value SW_Push -> KB
Connections:
- net VCC: now also SW2.2
- net at C29.2, SW1.1, U8.8 (RES): now also SW2.1
Changed lines of the file:
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@@
 	)
 	(junction
+		(at 31.75 392.43)
+		(diameter 0)
+		(color 0 0 0 0)
+	)
+	(junction
 		(at 33.02 40.64)
 		(diameter 0)
@@
 	)
 	(junction
+		(at 31.75 367.03)
+		(diameter 0)
+		(color 0 0 0 0)
+	)
+	(junction
 		(at 436.88 255.27)
 		(diameter 0)
@@
 	(wire
 		(pts
+			(xy 24.13 382.27) (xy 24.13 367.03)
+		)
+		(stroke
+			(width 0)
+			(type default)
+		)
+	)
+	(wire
+		(pts
 			(xy 457.2 243.84) (xy 457.2 250.19)
 		)
@@
 		)
 	)
+	(wire
+		(pts
+			(xy 24.13 367.03) (xy 31.75 367.03)
+		)
+		(stroke
+			(width 0)
+			(type default)
+		)
+	)
 	(bus
 		(pts
@@
 	(wire
 		(pts
+			(xy 24.13 392.43) (xy 31.75 392.43)
+		)
+		(stroke
+			(width 0)
+			(type default)
+		)
+	)
+	(wire
+		(pts
 			(xy 458.47 147.32) (xy 458.47 157.48)
 		)
@@
 		(fields_autoplaced yes)
 		(property "Reference" "SW1"
-			(at 33.02 386.08 90)
+			(at 33.02 386.0799 90)
 			(effects
 				(font
@@
 			)
 		)
-		(property "Value" "SW_Push"
-			(at 33.02 388.62 90)
+		(property "Value" "KB"
+			(at 33.02 388.6199 90)
 			(effects
 				(font
@@
 					(unit 1)
 				)
+			)
+		)
+	)
+	(symbol
+		(lib_id "Switch:SW_Push")
+		(at 24.13 387.35 90)
+		(unit 1)
+		(exclude_from_sim no)
+		(in_bom yes)
+		(on_board yes)
+		(dnp no)
+		(fields_autoplaced yes)
+		(property "Reference" "SW2"
+			(at 25.4 386.0799 90)
+			(effects
+				(font
+					(size 1.27 1.27)
+				)
+				(justify right)
+			)
+		)
+		(property "Value" "Old"
+			(at 25.4 388.6199 90)
+			(effects
+				(font
+					(size 1.27 1.27)
+				)
+				(justify right)
+			)
+		)
+		(property "Footprint" "SNES_Library:ResetSwitch"
+			(at 19.05 387.35 0)
+			(effects
+				(font
+					(size 1.27 1.27)
+				)
+				(hide yes)
+			)
+		)
+		(property "Datasheet" "~"
+			(at 19.05 387.35 0)
+			(effects
+				(font
+					(size 1.27 1.27)
+				)
+				(hide yes)
+			)
+		)
+		(property "Description" "Push button switch, generic, two pins"
+			(at 24.13 387.35 0)
+			(effects
+				(font
+					(size 1.27 1.27)
+				)
+				(hide yes)
+			)
+		)
+		(pin "1"
+		)
+		(pin "2"
+		)
+		(instances
+			(project "nonSNES"
+				(path "/d1480d56-b791-43e1-bd4c-b0c74bb0533d"
+					(reference "SW2")
+					(unit 1)
+				)
